File: ATtiny/ATtinyBoard/ATtinyBoard_2.sch (EAGLE design)
At the start: 19 parts, among them IC2 TINY13-20SU

Commit message: folder re-ordering
Parts:
- added R1, R2, R3: (no value), resistor:R-EU_M1406
Connections:
- removed net N$2: H3.P$1, H8.P$1, H9.P$1, IC2.PB4/PCINT4/ADC2
- removed net N$6: H10.P$1, H11.P$1, H2.P$1, IC2.PB3/PCINT3/CLKI/ADC3
- removed net N$7: H5.P$1, H6.P$1, H7.P$1, IC2.VCC, ISP/FTDI-CONNECTOR.4, JP2.2
- removed net N$8: H1.P$1, H12.P$1, H13.P$1, IC2.PB2/PCINT2/SCK/ADC1/T0, S3.1
- new net PB2: H1.P$1, H12.P$1, H13.P$1, IC2.PB2/PCINT2/SCK/ADC1/T0, R1.2, S3.1
- new net PB3: H10.P$1, H11.P$1, H2.P$1, IC2.PB3/PCINT3/CLKI/ADC3, R2.2
- new net PB4: H3.P$1, H8.P$1, H9.P$1, IC2.PB4/PCINT4/ADC2, R3.2
- new net VCC: H5.P$1, H6.P$1, H7.P$1, IC2.VCC, ISP/FTDI-CONNECTOR.4, JP2.2, R1.1, R2.1, R3.1
Other:
- moved on the sheet: JP2
Changed lines of the file:
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@@
 <part name="H14" library="LilyPad-Wearables" deviceset="SEW_HOLE-SMALL" device=""/>
 <part name="H15" library="LilyPad-Wearables" deviceset="SEW_HOLE-SMALL" device=""/>
+<part name="R1" library="resistor" deviceset="R-EU_" device="M1406"/>
+<part name="R2" library="resistor" deviceset="R-EU_" device="M1406"/>
+<part name="R3" library="resistor" deviceset="R-EU_" device="M1406"/>
 </parts>
 <sheets>
@@
 <instance part="ISP/FTDI-CONNECTOR" gate="G$1" x="5.08" y="81.28"/>
 <instance part="IC2" gate="G$1" x="101.6" y="71.12"/>
-<instance part="JP2" gate="G$1" x="38.1" y="119.38" rot="R270"/>
+<instance part="JP2" gate="G$1" x="38.1" y="124.46" rot="R270"/>
 <instance part="S3" gate="G$1" x="27.94" y="71.12" rot="R90"/>
 <instance part="H1" gate="G$1" x="38.1" y="43.18"/>
@@
 <instance part="H14" gate="G$1" x="76.2" y="38.1"/>
 <instance part="H15" gate="G$1" x="76.2" y="33.02"/>
+<instance part="R1" gate="G$1" x="12.7" y="60.96"/>
+<instance part="R2" gate="G$1" x="12.7" y="55.88"/>
+<instance part="R3" gate="G$1" x="12.7" y="50.8"/>
 </instances>
 <busses>
@@
 </segment>
 </net>
-<net name="N$7" class="0">
+<net name="VCC" class="0">
 <segment>
 <pinref part="IC2" gate="G$1" pin="VCC"/>
@@
 <wire x1="71.12" y1="83.82" x2="40.64" y2="83.82" width="0.1524" layer="91"/>
 <pinref part="JP2" gate="G$1" pin="2"/>
-<wire x1="40.64" y1="111.76" x2="40.64" y2="83.82" width="0.1524" layer="91"/>
+<wire x1="40.64" y1="116.84" x2="40.64" y2="83.82" width="0.1524" layer="91"/>
 <pinref part="ISP/FTDI-CONNECTOR" gate="G$1" pin="4"/>
 <wire x1="40.64" y1="83.82" x2="10.16" y2="83.82" width="0.1524" layer="91"/>
-<wire x1="71.12" y1="109.22" x2="71.12" y2="83.82" width="0.1524" layer="91"/>
+<wire x1="71.12" y1="109.22" x2="71.12" y2="96.52" width="0.1524" layer="91"/>
 <pinref part="H5" gate="G$1" pin="P$1"/>
 <pinref part="H6" gate="G$1" pin="P$1"/>
+<wire x1="71.12" y1="96.52" x2="71.12" y2="83.82" width="0.1524" layer="91"/>
 <wire x1="71.12" y1="109.22" x2="71.12" y2="114.3" width="0.1524" layer="91"/>
 <pinref part="H7" gate="G$1" pin="P$1"/>
 <wire x1="71.12" y1="114.3" x2="71.12" y2="119.38" width="0.1524" layer="91"/>
+<pinref part="R1" gate="G$1" pin="1"/>
+<pinref part="R2" gate="G$1" pin="1"/>
+<wire x1="7.62" y1="60.96" x2="7.62" y2="55.88" width="0.1524" layer="91"/>
+<pinref part="R3" gate="G$1" pin="1"/>
+<wire x1="7.62" y1="55.88" x2="7.62" y2="50.8" width="0.1524" layer="91"/>
+<wire x1="7.62" y1="50.8" x2="7.62" y2="27.94" width="0.1524" layer="91"/>
+<wire x1="7.62" y1="27.94" x2="129.54" y2="27.94" width="0.1524" layer="91"/>
+<wire x1="129.54" y1="27.94" x2="129.54" y2="96.52" width="0.1524" layer="91"/>
+<wire x1="129.54" y1="96.52" x2="71.12" y2="96.52" width="0.1524" layer="91"/>
+<label x="7.62" y="27.94" size="1.778" layer="95"/>
+<label x="124.46" y="27.94" size="1.778" layer="95"/>
+<label x="124.46" y="93.98" size="1.778" layer="95"/>
+<label x="71.12" y="104.14" size="1.778" layer="95"/>
 </segment>
 </net>
@@
 <pinref part="IC2" gate="G$1" pin="GND"/>
 <wire x1="81.28" y1="66.04" x2="73.66" y2="66.04" width="0.1524" layer="91"/>
-<wire x1="73.66" y1="66.04" x2="58.42" y2="66.04" width="0.1524" layer="91"/>
-<wire x1="58.42" y1="66.04" x2="58.42" y2="55.88" width="0.1524" layer="91"/>
-<label x="58.42" y="55.88" size="1.778" layer="95"/>
 <wire x1="73.66" y1="43.18" x2="73.66" y2="66.04" width="0.1524" layer="91"/>
 <pinref part="H4" gate="G$1" pin="P$1"/>
@@
 <pinref part="H15" gate="G$1" pin="P$1"/>
 <wire x1="73.66" y1="38.1" x2="73.66" y2="33.02" width="0.1524" layer="91"/>
-</segment>
-<segment>
+<wire x1="73.66" y1="66.04" x2="63.5" y2="66.04" width="0.1524" layer="91"/>
+<wire x1="63.5" y1="66.04" x2="63.5" y2="20.32" width="0.1524" layer="91"/>
+<wire x1="63.5" y1="20.32" x2="-2.54" y2="20.32" width="0.1524" layer="91"/>
+<wire x1="-2.54" y1="20.32" x2="-2.54" y2="96.52" width="0.1524" layer="91"/>
 <pinref part="ISP/FTDI-CONNECTOR" gate="G$1" pin="6"/>
 <wire x1="10.16" y1="88.9" x2="38.1" y2="88.9" width="0.1524" layer="91"/>
 <pinref part="JP2" gate="G$1" pin="1"/>
-<wire x1="38.1" y1="88.9" x2="38.1" y2="111.76" width="0.1524" layer="91"/>
+<wire x1="38.1" y1="88.9" x2="38.1" y2="116.84" width="0.1524" layer="91"/>
 <wire x1="10.16" y1="88.9" x2="10.16" y2="96.52" width="0.1524" layer="91"/>
-<wire x1="10.16" y1="96.52" x2="-10.16" y2="96.52" width="0.1524" layer="91"/>
-<wire x1="-10.16" y1="96.52" x2="-10.16" y2="86.36" width="0.1524" layer="91"/>
-<label x="-10.16" y="86.36" size="1.778" layer="95"/>
+<label x="33.02" y="88.9" size="1.778" layer="95"/>
+<wire x1="-2.54" y1="96.52" x2="10.16" y2="96.52" width="0.1524" layer="91"/>
+<label x="-2.54" y="20.32" size="1.778" layer="95"/>
+<label x="-2.54" y="96.52" size="1.778" layer="95"/>
+<label x="63.5" y="63.5" size="1.778" layer="95"/>
+<label x="73.66" y="45.72" size="1.778" layer="95"/>
 </segment>
 </net>
-<net name="N$2" class="0">
+<net name="PB4" class="0">
 <segment>
 <pinref part="IC2" gate="G$1" pin="PB4/PCINT4/ADC2"/>
 <wire x1="81.28" y1="71.12" x2="50.8" y2="71.12" width="0.1524" layer="91"/>
-<wire x1="50.8" y1="71.12" x2="50.8" y2="43.18" width="0.1524" layer="91"/>
+<wire x1="50.8" y1="71.12" x2="50.8" y2="50.8" width="0.1524" layer="91"/>
 <pinref part="H3" gate="G$1" pin="P$1"/>
 <pinref part="H8" gate="G$1" pin="P$1"/>
+<wire x1="50.8" y1="50.8" x2="50.8" y2="43.18" width="0.1524" layer="91"/>
 <wire x1="50.8" y1="43.18" x2="50.8" y2="38.1" width="0.1524" layer="91"/>
 <pinref part="H9" gate="G$1" pin="P$1"/>
 <wire x1="50.8" y1="38.1" x2="50.8" y2="33.02" width="0.1524" layer="91"/>
+<pinref part="R3" gate="G$1" pin="2"/>
+<wire x1="17.78" y1="50.8" x2="50.8" y2="50.8" width="0.1524" layer="91"/>
+<label x="50.8" y="45.72" size="1.778" layer="95"/>
 </segment>
 </net>
-<net name="N$6" class="0">
+<net name="PB3" class="0">
 <segment>
 <pinref part="IC2" gate="G$1" pin="PB3/PCINT3/CLKI/ADC3"/>
 <wire x1="81.28" y1="73.66" x2="43.18" y2="73.66" width="0.1524" layer="91"/>
-<wire x1="43.18" y1="73.66" x2="43.18" y2="43.18" width="0.1524" layer="91"/>
+<wire x1="43.18" y1="73.66" x2="43.18" y2="55.88" width="0.1524" layer="91"/>
 <pinref part="H2" gate="G$1" pin="P$1"/>
 <pinref part="H10" gate="G$1" pin="P$1"/>
+<wire x1="43.18" y1="55.88" x2="43.18" y2="43.18" width="0.1524" layer="91"/>
 <wire x1="43.18" y1="43.18" x2="43.18" y2="38.1" width="0.1524" layer="91"/>
 <pinref part="H11" gate="G$1" pin="P$1"/>
 <wire x1="43.18" y1="38.1" x2="43.18" y2="33.02" width="0.1524" layer="91"/>
+<pinref part="R2" gate="G$1" pin="2"/>
+<wire x1="17.78" y1="55.88" x2="43.18" y2="55.88" width="0.1524" layer="91"/>
+<label x="43.18" y="45.72" size="1.778" layer="95"/>
 </segment>
 </net>
-<net name="N$8" class="0">
+<net name="PB2" class="0">
 <segment>
 <pinref part="S3" gate="G$1" pin="1"/>
@@
 <pinref part="IC2" gate="G$1" pin="PB2/PCINT2/SCK/ADC1/T0"/>
 <wire x1="35.56" y1="76.2" x2="81.28" y2="76.2" width="0.1524" layer="91"/>
-<wire x1="35.56" y1="43.18" x2="35.56" y2="71.12" width="0.1524" layer="91"/>
+<wire x1="35.56" y1="43.18" x2="35.56" y2="60.96" width="0.1524" layer="91"/>
 <pinref part="H1" gate="G$1" pin="P$1"/>
 <pinref part="H12" gate="G$1" pin="P$1"/>
+<wire x1="35.56" y1="60.96" x2="35.56" y2="71.12" width="0.1524" layer="91"/>
 <wire x1="35.56" y1="43.18" x2="35.56" y2="38.1" width="0.1524" layer="91"/>
 <pinref part="H13" gate="G$1" pin="P$1"/>
 <wire x1="35.56" y1="38.1" x2="35.56" y2="33.02" width="0.1524" layer="91"/>
+<pinref part="R1" gate="G$1" pin="2"/>
+<wire x1="17.78" y1="60.96" x2="35.56" y2="60.96" width="0.1524" layer="91"/>
+<label x="35.56" y="45.72" size="1.778" layer="95"/>
 </segment>
 </net>
