File: projects/Gloves/xOSC Gloves/x-OSC Gloves_v2.sch (EAGLE design)
At the start: 58 parts

Commit message: MegaGlove final baord
Parts:
- removed PAD10, PAD11, PAD12, PAD13, PAD14, PAD15, PAD16, PAD17, PAD18, PAD19, PAD20, PAD21, PAD6, PAD7, PAD8, PAD9: (no value), wirepad:3,81/1,4
- added U$1, U$10, U$11, U$12, U$13, U$14, U$15, U$16, U$17, U$18, U$2, U$3, U$6, U$7, U$8, U$9: SNAP-PAD_7MM_ROUND, hannahsEagleLib:SNAP-PAD_7MM_ROUND
Connections:
- net GND: now also U$15.SNAPPAD, U$16.SNAPPAD, U$17.SNAPPAD, U$18.SNAPPAD; no longer PAD18.P, PAD19.P, PAD20.P, PAD21.P
- net N$12: now also U$8.SNAPPAD; no longer PAD10.P
- net N$13: now also U$9.SNAPPAD; no longer PAD9.P
- net N$14: now also U$10.SNAPPAD; no longer PAD8.P
- net N$15: now also U$11.SNAPPAD; no longer PAD7.P
- net N$16: now also U$12.SNAPPAD; no longer PAD6.P
- net N$23: now also U$13.SNAPPAD; no longer PAD16.P
- net N$24: now also U$14.SNAPPAD; no longer PAD17.P
- net N$4: now also U$1.SNAPPAD; no longer PAD15.P
- net N$6: now also U$2.SNAPPAD; no longer PAD14.P
- net N$7: now also U$3.SNAPPAD; no longer PAD13.P
- net N$8: now also U$6.SNAPPAD; no longer PAD12.P
- net N$9: now also U$7.SNAPPAD; no longer PAD11.P
Other:
- moved on the sheet: R1, R10, R11, R12, R13, R14, R19, R2, R3, R4, R5, R6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
