File: projects/Gloves/xOSC Gloves/x-OSC Gloves_v3.brd (EAGLE design)
At the start: 94 x 59.7 mm, 59 parts

Commit message: gloves updates
Parts:
- added U$17: MOTOR10MM, SparkFun-Electromechanical:VIBE-MOTOR-10MM
- added U$19, U$20: SNAP-PAD_7MM_ROUND, hannahsEagleLib:SNAP-PAD_7MM_RD
Connections:
- new net N$38: U$17.+, U$19.P$1
- new net N$46: U$17.-, U$20.P$1
Routing:
- net N$46: track 0.00 -> 15.7 mm
- net N$38: track 0.00 -> 7.14 mm
Other:
- board size 94 x 59.7 mm -> 108.1 x 59.7 mm
- board text added: "motor"
- board text added: "vibration"
Changed lines of the file:
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@@
 <layer number="116" name="Patch_BOT" color="9" fill="4" visible="no" active="yes"/>
 <layer number="121" name="_tsilk" color="7" fill="1" visible="yes" active="yes"/>
-<layer number="122" name="_bsilk" color="7" fill="1" visible="no" active="yes"/>
+<layer number="122" name="_bsilk" color="7" fill="1" visible="yes" active="yes"/>
 <layer number="125" name="_tNames" color="7" fill="1" visible="no" active="yes"/>
 <layer number="126" name="_bsilkInv" color="7" fill="1" visible="no" active="yes"/>
@@
 <text x="53" y="-1" size="1.778" layer="121">x-OSC flex</text>
 <dimension x1="48" y1="40.5" x2="48.69839375" y2="24.50743125" x3="49.0387" y3="16.714859375" textsize="1.778" layer="1" dtype="radius"/>
+<wire x1="96.749615625" y1="29.18858125" x2="105.858846875" y2="29.18858125" width="0.4064" layer="46" curve="-176.377619"/>
+<wire x1="105.91714375" y1="29.150190625" x2="106.767159375" y2="24.420946875" width="0.4064" layer="46" curve="55.04237"/>
+<wire x1="106.7893" y1="24.353275" x2="106.705171875" y2="13.14449375" width="0.4064" layer="46" curve="-91.769951"/>
+<wire x1="106.734996875" y1="13.192015625" x2="105.82951875" y2="9.866859375" width="0.4064" layer="46" curve="60.52427"/>
+<wire x1="105.81624375" y1="9.794071875" x2="96.442828125" y2="9.8453375" width="0.4064" layer="46" curve="-210.20711"/>
+<wire x1="96.389053125" y1="9.874021875" x2="95.240621875" y2="13.168275" width="0.4064" layer="46" curve="73.593687"/>
+<wire x1="95.230625" y1="13.1120625" x2="95.6410125" y2="24.61265625" width="0.4064" layer="46" curve="-93.311957"/>
+<wire x1="95.630084375" y1="24.66506875" x2="96.7644875" y2="29.2788125" width="0.4064" layer="46" curve="35.160963"/>
+<text x="100.84449375" y="14.8139125" size="1.778" layer="121" rot="R90">vibration</text>
+<text x="103.350690625" y="16.12805" size="1.778" layer="121" rot="R90">motor</text>
 </plain>
 <attributes>
@@
 </element>
 <element name="U$5" library="SparkFun-Connectors" package="USB-MINIB" value="USB-MINIB-5PIN" x="48" y="30" rot="R90"/>
+<element name="U$17" library="SparkFun-Electromechanical" package="VIBE-MOTOR-10MM" value="MOTOR10MM" x="102.48948125" y="18.09859375"/>
+<element name="U$19" library="hannahsEagleLib" package="SNAP-PAD_7MM_RD" value="SNAP-PAD_7MM_ROUND" x="101.161375" y="8.58050625"/>
+<element name="U$20" library="hannahsEagleLib" package="SNAP-PAD_7MM_RD" value="SNAP-PAD_7MM_ROUND" x="101.358640625" y="29.11891875"/>
 </elements>
 <signals>
@@
 <wire x1="42.613228125" y1="23.338003125" x2="42.613228125" y2="10.11543125" width="0.4064" layer="1"/>
 </signal>
+<signal name="N$38">
+<contactref element="U$19" pad="P$1"/>
+<contactref element="U$17" pad="+"/>
+<wire x1="97.48948125" y1="14.19859375" x2="101.161375" y2="10.5267" width="0.4064" layer="1" curve="-90"/>
+<wire x1="101.161375" y1="10.5267" x2="101.161375" y2="8.58050625" width="0.4064" layer="1"/>
+</signal>
+<signal name="N$46">
+<contactref element="U$17" pad="-"/>
+<contactref element="U$20" pad="P$1"/>
+<wire x1="101.358640625" y1="29.11891875" x2="101.358640625" y2="20.777753125" width="0.4064" layer="1"/>
+<wire x1="101.358640625" y1="20.777753125" x2="96.13948125" y2="15.55859375" width="0.4064" layer="1" curve="-90"/>
+</signal>
 </signals>
