File: projects/Gloves/xOSC Gloves/x-OSC Gloves_v3.sch (EAGLE design)
At the start: 59 parts

Commit message: gloves updates
Parts:
- added U$17: MOTOR10MM, SparkFun-Electromechanical:MOTOR10MM
- added U$19, U$20: SNAP-PAD_7MM_ROUND, hannahsEagleLib:SNAP-PAD_7MM_ROUND
Connections:
- new net N$38: U$17.+, U$19.SNAPPAD
- new net N$46: U$17.-, U$20.SNAPPAD
Changed lines of the file:
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@@
 <part name="TP22" library="testpad" deviceset="TP" device="TP20R"/>
 <part name="U$5" library="SparkFun-Connectors" deviceset="USB-MINIB" device="-5PIN"/>
+<part name="U$17" library="SparkFun-Electromechanical" deviceset="MOTOR" device="10MM"/>
+<part name="U$19" library="hannahsEagleLib" deviceset="SNAP-PAD_7MM_ROUND" device=""/>
+<part name="U$20" library="hannahsEagleLib" deviceset="SNAP-PAD_7MM_ROUND" device=""/>
 </parts>
 <sheets>
@@
 <instance part="TP22" gate="G$1" x="332.74" y="-12.7"/>
 <instance part="U$5" gate="G$1" x="208.28" y="-76.2" rot="R270"/>
+<instance part="U$17" gate="G$1" x="157.48" y="12.7" rot="R90"/>
+<instance part="U$19" gate="G$1" x="137.16" y="12.7" rot="R90"/>
+<instance part="U$20" gate="G$1" x="177.8" y="12.7" rot="R270"/>
 </instances>
 <busses>
@@
 </segment>
 </net>
+<net name="N$38" class="0">
+<segment>
+<pinref part="U$19" gate="G$1" pin="SNAPPAD"/>
+<pinref part="U$17" gate="G$1" pin="+"/>
+<wire x1="149.86" y1="12.7" x2="152.4" y2="12.7" width="0.1524" layer="91"/>
+</segment>
+</net>
+<net name="N$46" class="0">
+<segment>
+<pinref part="U$17" gate="G$1" pin="-"/>
+<pinref part="U$20" gate="G$1" pin="SNAPPAD"/>
+<wire x1="162.56" y1="12.7" x2="165.1" y2="12.7" width="0.1524" layer="91"/>
+</segment>
+</net>
