File: projects/Gloves/xOSC Gloves/x-OSC Gloves_v4.sch (EAGLE design)
At the start: 57 parts

Commit message: gloves updates
Parts:
- removed LED2: F50360, led:F50360
- removed TP11, TP12, TP13, TP14, TP15, TP16, TP17, TP18, TP19, TP20: TPTP20R, testpad:TPTP20R
- removed U$12: SNAP-PAD_7MM_ROUND, hannahsEagleLib:SNAP-PAD_7MM_ROUND
- added R18: (no value), SparkFun-Passives:RESISTOR0805-RES
- added TP21, TP22: TPTP20R, testpad:TPTP20R
- added U$19, U$20, U$21: SNAP-PAD_7MM_ROUND, hannahsEagleLib:SNAP-PAD_7MM_ROUND
- added U$5: USB-MINIB-5PIN, SparkFun-Connectors:USB-MINIB-5PIN
- U$17: value SNAP-PAD_7MM_ROUND -> MOTOR10MM; device hannahsEagleLib:SNAP-PAD_7MM_ROUND -> SparkFun-Electromechanical:MOTOR10MM
Connections:
- removed net N$26: TP11.TP, U$4.OUT14
- removed net N$29: TP12.TP, U$4.OUT13
- removed net N$30: TP13.TP, U$4.OUT12
- removed net N$31: TP14.TP, U$4.OUT11
- removed net N$32: TP15.TP, U$4.OUT10
- new net N$33: U$4.VBATT, U$5.VBUS
- new net N$38: U$17.+, U$19.SNAPPAD
- new net N$40: R18.2, U$21.SNAPPAD, U$4.IN1
- new net N$46: U$17.-, U$20.SNAPPAD
- net GND: now also TP22.TP, U$5.GND; no longer LED2.BC, LED2.GC, LED2.RC, TP16.TP, TP17.TP, TP18.TP, TP19.TP, TP20.TP, U$17.SNAPPAD
- net N$1: no longer LED2.BA
- net N$16: now also TP21.TP; no longer U$12.SNAPPAD
- net N$17: no longer LED2.RA
- net N$2: no longer LED2.GA
- net VDD: now also R18.1
