File: projects/Gloves/xOSC Gloves/x-OSC Gloves_v5.sch (EAGLE design)
At the start: 57 parts

Commit message: gloves updates
Parts:
- removed LED1: F50360, led:F50360
- removed TP11, TP12, TP13, TP14, TP15, TP16, TP17, TP18, TP19, TP20: TPTP20R, testpad:TPTP20R
- removed U$13, U$14, U$15, U$16, U$18: SNAP-PAD_7MM_ROUND, hannahsEagleLib:SNAP-PAD_7MM_ROUND
- added LED2: LED-TRICOLOR-5050NO_IC, SparkFun-LED:LED-TRICOLOR-5050NO_IC
- added TP22: TPTP20R, testpad:TPTP20R
- added U$17: MOTOR10MM, SparkFun-Electromechanical:MOTOR10MM
- added U$21: SNAP-PAD_7MM_ROUND, hannahsEagleLib:SNAP-PAD_7MM_ROUND
- added U$5: USB-MINIB-5PIN, SparkFun-Connectors:USB-MINIB-5PIN
- U$12: value SNAP-PAD_7MM_ROUND -> MOTOR10MM; device hannahsEagleLib:SNAP-PAD_7MM_ROUND -> SparkFun-Electromechanical:MOTOR10MM
Connections:
- removed net N$26: TP11.TP, U$4.OUT14
- removed net N$29: TP12.TP, U$4.OUT13
- removed net N$30: TP13.TP, U$4.OUT12
- removed net N$31: TP14.TP, U$4.OUT11
- removed net N$32: TP15.TP, U$4.OUT10
- new net N$33: U$4.VBATT, U$5.VBUS
- net GND: now also LED2.BLU-C, LED2.GRN-C, LED2.RED-C, TP22.TP, U$12.-, U$17.-, U$5.GND; no longer LED1.BC, LED1.GC, LED1.RC, TP16.TP, TP17.TP, TP18.TP, TP19.TP, TP20.TP, U$15.SNAPPAD, U$16.SNAPPAD, U$18.SNAPPAD
- net N$1: now also LED2.GRN-A, R16.2; no longer LED1.BA, R15.2
- net N$16: now also TP21.TP; no longer U$12.SNAPPAD
- net N$17: now also LED2.BLU-A; no longer LED1.RA
- net N$2: now also LED2.RED-A, R15.2; no longer LED1.GA, R16.2
- net N$23: now also U$17.+; no longer U$13.SNAPPAD
- net N$24: now also U$12.+; no longer U$14.SNAPPAD
- net N$25: now also U$4.OUT3; no longer U$4.OUT1
- net N$3: now also U$4.OUT2; no longer U$4.OUT3
- net N$40: now also U$21.SNAPPAD; no longer TP21.TP
- net N$5: now also U$4.OUT1; no longer U$4.OUT2
Other:
- moved on the sheet: TP21
