File: projects/Gloves/xOSC Gloves/x-OSC Gloves_v6.brd (EAGLE design)
At the start: 123.5 x 80 mm, 46 parts

Commit message: final stulpe
Parts:
- added S1: (no value), SparkFun-Electromechanical:SWITCH-SPST-SMD-A
- moved U$8 63.1 mm to (20.1, 44.8)
- moved U$3 63.1 mm to (79.7, 24.8)
- moved U$10 61.0 mm to (20.0, 24.8)
- moved U$1 61.0 mm to (80.0, 45.2)
- moved U$6 20.3 mm to (80.0, 14.6)
- moved U$7 20.0 mm to (20.0, 54.7)
- moved U$9 10.2 mm to (20.0, 35.2)
- moved U$2 9.89 mm to (80.1, 35.1)
- moved R6 9.80 mm to (68.7, 41.2), turned to 180 degrees
- moved R8 9.74 mm to (68.6, 36.2), turned to 180 degrees
- moved R9 9.64 mm to (68.6, 32.4), turned to 180 degrees
- moved R7 9.55 mm to (68.5, 37.9), turned to 180 degrees
- moved R5 8.82 mm to (67.8, 42.9), turned to 180 degrees
- moved U$5 5.81 mm to (47.2, 12.0)
- moved TP6 4.83 mm to (47.5, 21.9)
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Connections:
- new net N$26: S1.1, U$5.GND
- net GND: now also S1.2, U$17.+; no longer U$17.-, U$5.GND
- net N$23: now also U$17.-; no longer U$17.+
Routing:
- net GND: track 166.5 -> 232.6 mm
- net VDD: track 39.9 -> 77.4 mm, vias 0 -> 2
- net N$4: track 54.9 -> 23.1 mm
- net N$12: track 27.4 -> 50.5 mm
- net N$7: track 55.8 -> 34.9 mm
- net N$14: track 32.6 -> 50.9 mm
- net N$8: track 24.8 -> 43.0 mm
- net N$26: track 0.00 -> 15.9 mm
- net N$13: track 56.4 -> 48.9 mm, vias 1 -> 0
- net N$15: track 59.6 -> 52.4 mm
- net N$6: track 22.9 -> 28.9 mm
- net N$9: track 55.5 -> 50.2 mm, vias 1 -> 0
- net N$23: track 56.7 -> 54.3 mm
- net N$33: track 13.0 -> 11.4 mm
- net N$24: track 28.1 -> 29.6 mm
Other:
- outline, holes or cut-outs redrawn
- board text added: "left"
- board text added: "off"
- board text added: "on"
- board text added: "right"
