File: projects/Gloves/xOSC Gloves/x-OSC Gloves_v6.sch (EAGLE design)
At the start: 58 parts

Commit message: gloves updates
Parts:
- removed LED1: F50360, led:F50360
- removed TP11, TP12, TP13, TP14, TP15, TP16, TP17, TP18, TP19, TP20: TPTP20R, testpad:TPTP20R
- removed U$13, U$14, U$15, U$16, U$18: SNAP-PAD_7MM_ROUND, hannahsEagleLib:SNAP-PAD_7MM_ROUND
- added LED2: LED-TRICOLOR-5050NO_IC, SparkFun-LED:LED-TRICOLOR-5050NO_IC
- added U$17: MOTOR10MM, SparkFun-Electromechanical:MOTOR10MM
- added U$21: SNAP-PAD_7MM_ROUND, hannahsEagleLib:SNAP-PAD_7MM_ROUND
- added U$5: USB-MINIB-5PIN, SparkFun-Connectors:USB-MINIB-5PIN
- U$12: value SNAP-PAD_7MM_ROUND -> MOTOR10MM; device hannahsEagleLib:SNAP-PAD_7MM_ROUND -> SparkFun-Electromechanical:MOTOR10MM
Connections:
- removed net N$26: TP11.TP, U$4.OUT14
- removed net N$29: TP12.TP, U$4.OUT13
- removed net N$30: TP13.TP, U$4.OUT12
- removed net N$31: TP14.TP, U$4.OUT11
- removed net N$32: TP15.TP, U$4.OUT10
- new net N$33: U$4.VBATT, U$5.VBUS
- net GND: now also LED2.BLU-C, LED2.GRN-C, LED2.RED-C, U$12.-, U$17.-, U$5.GND; no longer LED1.BC, LED1.GC, LED1.RC, TP16.TP, TP17.TP, TP18.TP, TP19.TP, TP20.TP, U$15.SNAPPAD, U$16.SNAPPAD, U$18.SNAPPAD
- net N$1: now also LED2.GRN-A, R16.2; no longer LED1.BA, R15.2
- net N$16: now also TP21.TP; no longer U$12.SNAPPAD
- net N$17: now also LED2.BLU-A; no longer LED1.RA
- net N$2: now also LED2.RED-A, R15.2; no longer LED1.GA, R16.2
- net N$23: now also U$17.+; no longer U$13.SNAPPAD
- net N$24: now also U$12.+; no longer U$14.SNAPPAD
- net N$25: now also U$4.OUT3; no longer U$4.OUT1
- net N$3: now also U$4.OUT2; no longer U$4.OUT3
- net N$40: now also U$21.SNAPPAD; no longer TP21.TP
- net N$5: now also U$4.OUT1; no longer U$4.OUT2
Other:
- moved on the sheet: TP21

Commit message: final stulpe
Parts:
- added S1: (no value), SparkFun-Electromechanical:SWITCH-SPDT-SMD-A
Connections:
- new net N$26: S1.O, U$5.GND
- net GND: now also S1.P, U$17.+; no longer U$17.-, U$5.GND
- net N$23: now also U$17.-; no longer U$17.+
Other:
- moved on the sheet: U$17
Changed lines of the file:
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@@
 <part name="U$12" library="SparkFun-Electromechanical" deviceset="MOTOR" device="10MM"/>
 <part name="LED2" library="SparkFun-LED" deviceset="LED-TRICOLOR-5050" device="NO_IC"/>
+<part name="S1" library="SparkFun-Electromechanical" deviceset="SWITCH-SPDT" device="-SMD-A"/>
 </parts>
 <sheets>
@@
 <instance part="R18" gate="G$1" x="40.64" y="-27.94"/>
 <instance part="TP22" gate="G$1" x="332.74" y="-12.7"/>
-<instance part="U$5" gate="G$1" x="208.28" y="-76.2" rot="R270"/>
-<instance part="U$17" gate="G$1" x="238.76" y="-5.08" rot="R180"/>
+<instance part="U$5" gate="G$1" x="236.22" y="-76.2" rot="R270"/>
+<instance part="U$17" gate="G$1" x="238.76" y="-5.08"/>
 <instance part="U$21" gate="G$1" x="48.26" y="2.54"/>
 <instance part="U$12" gate="G$1" x="243.84" y="-5.08" rot="R180"/>
 <instance part="LED2" gate="D1" x="203.2" y="7.62" rot="R270"/>
+<instance part="S1" gate="1" x="210.82" y="-73.66"/>
 </instances>
 <busses>
@@
 <wire x1="215.9" y1="-33.02" x2="231.14" y2="-33.02" width="0.1524" layer="91"/>
 <pinref part="TP22" gate="G$1" pin="TP"/>
-<pinref part="U$12" gate="G$1" pin="-"/>
-<pinref part="U$17" gate="G$1" pin="-"/>
 <wire x1="231.14" y1="-33.02" x2="251.46" y2="-33.02" width="0.1524" layer="91"/>
-<wire x1="243.84" y1="0" x2="238.76" y2="0" width="0.1524" layer="91"/>
-<wire x1="238.76" y1="0" x2="231.14" y2="0" width="0.1524" layer="91"/>
 <wire x1="231.14" y1="0" x2="231.14" y2="-33.02" width="0.1524" layer="91"/>
 <pinref part="LED2" gate="D1" pin="RED-C"/>
@@
 <wire x1="205.74" y1="22.86" x2="215.9" y2="22.86" width="0.1524" layer="91"/>
 <wire x1="215.9" y1="22.86" x2="215.9" y2="-33.02" width="0.1524" layer="91"/>
+<pinref part="U$17" gate="G$1" pin="+"/>
+<wire x1="231.14" y1="0" x2="238.76" y2="0" width="0.1524" layer="91"/>
+<pinref part="U$12" gate="G$1" pin="-"/>
+<wire x1="238.76" y1="0" x2="243.84" y2="0" width="0.1524" layer="91"/>
 </segment>
 <segment>
@@
 <wire x1="139.7" y1="-83.82" x2="139.7" y2="-88.9" width="0.1524" layer="91"/>
 <label x="139.7" y="-88.9" size="1.778" layer="95"/>
-<pinref part="U$5" gate="G$1" pin="GND"/>
-<wire x1="208.28" y1="-73.66" x2="208.28" y2="-71.12" width="0.1524" layer="91"/>
-<wire x1="208.28" y1="-71.12" x2="195.58" y2="-71.12" width="0.1524" layer="91"/>
+<pinref part="S1" gate="1" pin="P"/>
+<wire x1="195.58" y1="-71.12" x2="208.28" y2="-71.12" width="0.1524" layer="91"/>
+<wire x1="208.28" y1="-71.12" x2="208.28" y2="-73.66" width="0.1524" layer="91"/>
 </segment>
 </net>
@@
 <pinref part="U$4" gate="G$1" pin="OUT15"/>
 <wire x1="238.76" y1="-63.5" x2="187.96" y2="-63.5" width="0.1524" layer="91"/>
-<pinref part="U$17" gate="G$1" pin="+"/>
+<pinref part="U$17" gate="G$1" pin="-"/>
 <wire x1="238.76" y1="-10.16" x2="238.76" y2="-63.5" width="0.1524" layer="91"/>
 </segment>
@@
 <pinref part="U$4" gate="G$1" pin="VBATT"/>
 <pinref part="U$5" gate="G$1" pin="VBUS"/>
-<wire x1="187.96" y1="-68.58" x2="218.44" y2="-68.58" width="0.1524" layer="91"/>
-<wire x1="218.44" y1="-68.58" x2="218.44" y2="-73.66" width="0.1524" layer="91"/>
+<wire x1="187.96" y1="-68.58" x2="246.38" y2="-68.58" width="0.1524" layer="91"/>
+<wire x1="246.38" y1="-68.58" x2="246.38" y2="-73.66" width="0.1524" layer="91"/>
 </segment>
 </net>
@@
 </segment>
 </net>
+<net name="N$26" class="0">
+<segment>
+<pinref part="U$5" gate="G$1" pin="GND"/>
+<wire x1="236.22" y1="-73.66" x2="236.22" y2="-71.12" width="0.1524" layer="91"/>
+<wire x1="236.22" y1="-71.12" x2="215.9" y2="-71.12" width="0.1524" layer="91"/>
+<pinref part="S1" gate="1" pin="O"/>
+</segment>
+</net>
