File: projects/Hahnentrittstulpe/Hahnentrittstulpe.brd (EAGLE design)
At the start: 100 x 80 mm, 10 parts, among them IC1 TINY13-20SU

Commit message: final stulpe
Routing:
- net N$5: track 125.7 -> 127.9 mm
- net N$9: track 117.7 -> 118.4 mm
Other:
- board text removed: "Stulpe"
