File: projects/LeatherSynth/LeatherSynth.brd (EAGLE design)
At the start: 100 x 80 mm, 54 parts, among them IC1 TL072P, Q1 BC557, T1 BC547, T2 BC547, T3 BC547, T4 BC547, T5 BC547, X1 22-23-2021

Commit message: 808
Parts:
- added R28: 50K, pot:3223J
- added R29: 500K, pot:3223J
- added R30: 10K, pot:3223J
- added R31: 100K, eagle-ltspice:R2010
- added R32: 100K, pot:3223J
- added R33: 10K, eagle-ltspice:R2010
- added U$1: (no value), hannah:LEATHERSYNTH
- added U$2: (no value), hannah:LEATHERSYNTH2
- added U$3: AYZ0202, SparkFun-Electromechanical:AYZ0202
- added X2: 22-23-2021, con-molex:22-23-2021
- moved S1 352.7 mm to (50.0, 79.2), turned to 90 degrees
- moved C9 323.3 mm to (76.7, 61.5)
- moved C7 313.9 mm to (88.1, 52.8)
- moved C8 313.8 mm to (79.0, 53.6)
- moved C13 298.5 mm to (51.3, 28.4)
- moved C10 298.4 mm to (24.1, 57.1)
- moved C12 296.5 mm to (22.9, 48.3)
- moved C6 296.3 mm to (70.6, 47.0)
- moved X1 296.1 mm to (1.78, 45.7), turned to 90 degrees
- moved C3 294.5 mm to (90.9, 46.2)
- moved C4 293.8 mm to (80.3, 47.0)
- moved C11 289.8 mm to (13.7, 49.0)
- moved C1 286.9 mm to (70.1, 54.1)
- moved SV1 283.0 mm to (51.6, 2.03)
- moved C2 280.0 mm to (61.7, 47.0), turned to 180 degrees
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Connections:
- removed net N$19: SV1.2
- removed net N$23: T2.1
- removed net N$25: D1.C
- removed net N$45: S1.2
- removed net N$53: C12.1, C4.1
- removed net V+: IC1.8
- removed net V-: IC1.4
- new net +9V: IC1.8, LED1.A, R19.2, R27.2, R31.2, S1.2, SV1.3
- new net -9V: IC1.4, R33.1, R5.1, SV1.1
- new net B2: T5.3
- new net N$1: R12.1, R13.2
- new net N$14: C11.1, R11.2, R2.1
- new net N$6: C3.1, R29.2
- new net N$8: R16.2, R30.3
- new net N$9: C12.1, C4.1, R16.1, R30.1, R30.2
- net GND: now also C2.2, D1.C, R11.1, R18.1, R24.1, R25.1, R28.2, R3.1, R32.1, R4.1, R8.1, T2.1, U$3.2, X2.2; no longer SV1.1
- net N$10: now also R32.3
- net N$11: now also R32.2
- net N$13: now also R25.2, T5.2
- net N$15: now also LED1.C, R33.2; no longer C11.1, R2.1
- net N$16: now also C2.1, R5.2
- net N$17: now also SV1.2, U$3.1; no longer SV1.3
- net N$18: now also R13.1
- net N$20: now also R7.1
- net N$21: now also R28.3
- net N$24: now also R26.1
- net N$26: now also R22.2
- net N$34: now also R3.2, R6.2
- net N$38: now also R6.1
- net N$39: now also R14.2, R31.1
- net N$4: now also R21.2, R29.1, R9.1
- net N$42: now also R14.1, R17.2
- net N$43: now also R17.1
- net N$47: now also R24.2
- net N$48: now also R20.2
- net N$49: now also R18.2, R20.1
- net N$5: now also R8.2
- net N$52: now also X2.1
- net N$7: now also R26.2
Other:
- board size 100 x 80 mm -> 100.3 x 80.3 mm
